File: Schematic/KiCAD/ff-osd-adapter.kicad_pcb (KiCad board)
At the start: 2 copper layers, 31.5 x 66.5 mm, 8 parts, among them J1 GOTEK, J2 Amiga_Video, J3 Programming, J5 Amiga_Keyboard, U1 BluePill_STM32F103C

Commit message: Cosmetic Changes
Other:
- board text added: "RCEU1520 - FlashFloppy OSD Adapter v1.0 Copyright (c) 2020 Tomse @ http://retro-commodore.eu"
- board text removed: "FlashFloppy OSD Adapter v1.0 by Tomse @ http://retro-commodore.eu 2020"
Changed lines of the file:
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@@
   )
   (page A4)
+  (title_block
+    (title "RCEU1520 - FlashFloppy OSD Adapter")
+    (date 2020-04-06)
+    (rev 1)
+    (comment 3 "by Tomse in 2020")
+    (comment 4 http://retro-commodore.eu)
+  )
   (layers
     (0 F.Cu signal)
@@
       (drillshape 0)
       (scaleselection 1)
-      (outputdirectory "FlashFloppy-OSD-Adapter/"))
+      (outputdirectory "RCEU1520-FlashFloppy-OSD-Adapter/"))
   )
   (net 0 "")
@@
     )
   )
-  (gr_text "FlashFloppy OSD Adapter v1.0\nby Tomse @ http://retro-commodore.eu\n2020" (at 103.5 90.5 90) (layer B.Cu)
+  (gr_text "RCEU1520 - FlashFloppy OSD Adapter v1.0\nCopyright (c) 2020 \nTomse @ http://retro-commodore.eu\n\n" (at 103.5 90.5 90) (layer B.Cu)
     (effects (font (size 1.2 1.2) (thickness 0.2)) (justify mirror))
   )

Commit message: Cosmetic changes/corrections
Other:
- board text added: "USB Port side here"
Changed lines of the file:
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@@
   (general
     (thickness 1.6)
-    (drawings 21)
+    (drawings 22)
     (tracks 43)
     (zones 0)
@@
     )
   )
+  (gr_text "USB Port\nside here" (at 103 70.5) (layer F.SilkS)
+    (effects (font (size 1.5 1.5) (thickness 0.3)))
+  )
   (gr_text "RCEU1520 - FlashFloppy OSD Adapter v1.0\nCopyright (c) 2020 \nTomse @ http://retro-commodore.eu\n\n" (at 103.5 90.5 90) (layer B.Cu)
     (effects (font (size 1.2 1.2) (thickness 0.2)) (justify mirror))
@@
     (effects (font (size 1 1) (thickness 0.15)))
   )
-  (gr_text "3v3\n" (at 86.5 118.5 270) (layer F.SilkS)
+  (gr_text "3v3\n" (at 86.5 113.75 270) (layer F.SilkS)
     (effects (font (size 1 1) (thickness 0.15)))
   )
-  (gr_text "GND\n" (at 86.5 114 270) (layer F.SilkS)
+  (gr_text "GND\n" (at 86.5 118 270) (layer F.SilkS)
     (effects (font (size 1 1) (thickness 0.15)))
   )

Commit message: v1.1 - added support for Amiga Keyboard disk change control
Parts:
- added KeyCtrl: Amiga_Key_Input_To_FF, Jumper:SolderJumper-2_P1.3mm_Bridged_RoundedPad1.0x1.5mm, F.Cu at (89.0, 101.2)
- renumbered J2 to J1, J1 to J2, J5 to J4
Routing:
- net Net-(JP1-Pad2): track 0.00 -> 25.3 mm
- net Net-(JP1-Pad1): track 0.00 -> 24.8 mm
Other:
- board text added: "RCEU1520 - FlashFloppy OSD Adapter v1.1 Copyright (c) 2020 Tomse @ http://retro-commodore.eu"
- board text removed: "RCEU1520 - FlashFloppy OSD Adapter v1.0 Copyright (c) 2020 Tomse @ http://retro-commodore.eu"
